File: 8259.kicad_sch (KiCad schematic)
At the start: 7 parts, among them J61 Conn_01x04, SW61 SW_Push, U61 8259, U62 PAL16L8, U63 PAL16L8

Commit message: Added bullet 6
Parts:
- added R62: 10K, symbol Device:R
Connections:
- net VCC: now also R62.2; no longer U61.16 (~{SP}/~{EN})
- net Wait: no longer names the net of U61.1 (~{CS}), U62.19 (IO1)
- new net: R62.1, U61.16 (~{SP}/~{EN})
Changed lines of the file:
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@@
+    (stroke (width 0) (type default) (color 0 0 0 0))
+  )
+  (wire (pts (xy 109.982 96.52) (xy 112.148 96.52))
     (stroke (width 0) (type default) (color 0 0 0 0))
   )
@@
   )
   (wire (pts (xy 67.818 129.54) (xy 67.818 156.972))
+    (stroke (width 0) (type default) (color 0 0 0 0))
+  )
+  (wire (pts (xy 112.148 96.52) (xy 112.148 96.5193))
     (stroke (width 0) (type default) (color 0 0 0 0))
   )
@@
     (effects (font (size 1.27 1.27)) (justify left))
   )
+  (hierarchical_label "VCC" (shape input) (at 119.768 96.5193 90)
+    (effects (font (size 1.27 1.27)) (justify left))
+  )
   (hierarchical_label "VCC" (shape input) (at 55.118 106.68 90)
     (effects (font (size 1.27 1.27)) (justify left))
   )
-  (hierarchical_label "VCC" (shape input) (at 109.982 96.52 0)
-    (effects (font (size 1.27 1.27)) (justify left))
-  )
   (hierarchical_label "IR1" (shape input) (at 109.982 78.74 0)
     (effects (font (size 1.27 1.27)) (justify left))
@@
   (hierarchical_label "IR2" (shape input) (at 109.982 76.2 0)
     (effects (font (size 1.27 1.27)) (justify left))
-  )
-  (hierarchical_label "Wait" (shape input) (at 67.8291 91.44 180)
-    (effects (font (size 1.27 1.27)) (justify right))
   )
   (hierarchical_label "RD" (shape input) (at 79.502 96.52 180)
@@
       (effects (font (size 1.27 1.27)) hide)
     )
+    (pin "1")
+    (pin "2")
+  )
+  (symbol (lib_id "Device:R") (at 115.958 96.5193 90) (unit 1)
+    (in_bom yes) (on_board yes) (fields_autoplaced)
+    (property "Reference" "R62" (id 0) (at 115.958 90.17 90))
+    (property "Value" "10K" (id 1) (at 115.958 92.71 90))
+    (property "Footprint" "" (id 2) (at 115.958 98.2973 90)
+      (effects (font (size 1.27 1.27)) hide)
+    )
+    (property "Datasheet" "~" (id 3) (at 115.958 96.5193 0)
+      (effects (font (size 1.27 1.27)) hide)
+    )
