File: 8259.kicad_sch (KiCad schematic)
At the start: 11 parts, among them J61 Conn_01x04, SW61 SW_Push, U61 8259, U62 PAL16L8, U63 74LVC2G32, U64 74LVC2G32, U65 74LVC2G32

Commit message: yes
Parts:
- U63, U64, U65: footprint Package_SO:SSOP-8_2.95x2.8mm_P0.65mm -> (none)
Changed lines of the file:
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@@
     (property "Reference" "U63" (id 0) (at 42.991 185.7221 0))
     (property "Value" "74LVC2G32" (id 1) (at 42.991 188.2621 0))
-    (property "Footprint" "Package_SO:SSOP-8_2.95x2.8mm_P0.65mm" (id 2) (at 43.626 193.8501 0)
+    (property "Footprint" "" (id 2) (at 43.626 193.8501 0)
       (effects (font (size 1.27 1.27)) hide)
     )
@@
     (property "Reference" "U64" (id 0) (at 43.372 206.8041 0))
     (property "Value" "74LVC2G32" (id 1) (at 43.372 209.3441 0))
-    (property "Footprint" "Package_SO:SSOP-8_2.95x2.8mm_P0.65mm" (id 2) (at 43.372 202.4861 0)
+    (property "Footprint" "" (id 2) (at 43.372 202.4861 0)
       (effects (font (size 1.27 1.27)) hide)
     )
@@
     (property "Reference" "U65" (id 0) (at 56.961 189.5321 0))
     (property "Value" "74LVC2G32" (id 1) (at 56.961 192.0721 0))
-    (property "Footprint" "Package_SO:SSOP-8_2.95x2.8mm_P0.65mm" (id 2) (at 57.596 197.9141 0)
+    (property "Footprint" "" (id 2) (at 57.596 197.9141 0)
       (effects (font (size 1.27 1.27)) hide)
     )

Commit message: Finished
Parts:
- U63, U64, U65: footprint (none) -> Package_DIP:DIP-8_W7.62mm
Changed lines of the file:
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@@
     (property "Reference" "U63" (id 0) (at 42.991 185.7221 0))
     (property "Value" "74LVC2G32" (id 1) (at 42.991 188.2621 0))
-    (property "Footprint" "" (id 2) (at 43.626 193.8501 0)
+    (property "Footprint" "Package_DIP:DIP-8_W7.62mm" (id 2) (at 43.626 193.8501 0)
       (effects (font (size 1.27 1.27)) hide)
     )
@@
     (property "Reference" "U64" (id 0) (at 43.372 206.8041 0))
     (property "Value" "74LVC2G32" (id 1) (at 43.372 209.3441 0))
-    (property "Footprint" "" (id 2) (at 43.372 202.4861 0)
+    (property "Footprint" "Package_DIP:DIP-8_W7.62mm" (id 2) (at 43.372 202.4861 0)
       (effects (font (size 1.27 1.27)) hide)
     )
@@
     (property "Reference" "U65" (id 0) (at 56.961 189.5321 0))
     (property "Value" "74LVC2G32" (id 1) (at 56.961 192.0721 0))
-    (property "Footprint" "" (id 2) (at 57.596 197.9141 0)
+    (property "Footprint" "Package_DIP:DIP-8_W7.62mm" (id 2) (at 57.596 197.9141 0)
       (effects (font (size 1.27 1.27)) hide)
     )
