File: 8086 Bullet One.kicad_sch (KiCad schematic)
At the start: 13 parts, among them J1 Conn_01x20, J2 Conn_01x16, J3 Conn_01x03, SW0 SW_Push, U1 8086_Min_Mode, U2 74AHC373, U3 74AHC373, U4 74AHC373, U5 74LS245, U6 74LS245, U7 74LS244

Commit message: Added bullet 6
Connections:
- net HLDA: no longer names the net of U1.30 (HLDA)
- net HOLD: no longer names the net of U1.31 (HOLD)
- no-connect marks 12 -> 14
Changed lines of the file:
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@@
   (no_connect (at 134.62 151.13))
   (no_connect (at 134.62 153.67))
+  (no_connect (at 69.85 82.55))
+  (no_connect (at 69.85 77.47))
   (no_connect (at 180.34 146.05))
   (no_connect (at 205.74 140.97))
@@
     (stroke (width 0) (type default) (color 0 0 0 0))
   )
-  (wire (pts (xy 141.2951 146.05) (xy 142.748 146.05))
+  (wire (pts (xy 141.2951 146.05) (xy 144.526 146.05))
     (stroke (width 0) (type default) (color 0 0 0 0))
   )
@@
     (stroke (width 0) (type default) (color 0 0 0 0))
   )
-  (wire (pts (xy 141.986 143.51) (xy 142.748 143.51))
+  (wire (pts (xy 141.986 143.51) (xy 144.272 143.51))
     (stroke (width 0) (type default) (color 0 0 0 0))
   )
@@
     (stroke (width 0) (type default) (color 0 0 0 0))
   )
+  (wire (pts (xy 105.41 115.824) (xy 105.41 110.49))
+    (stroke (width 0) (type default) (color 0 0 0 0))
+  )
   (wire (pts (xy 105.41 107.95) (xy 106.68 107.95))
     (stroke (width 0) (type default) (color 0 0 0 0))
@@
     (stroke (width 0) (type default) (color 0 0 0 0))
   )
-  (wire (pts (xy 140.3761 148.59) (xy 143.002 148.59))
+  (wire (pts (xy 140.3761 148.59) (xy 144.526 148.59))
     (stroke (width 0) (type default) (color 0 0 0 0))
   )
@@
     (effects (font (size 1.27 1.27)) (justify left bottom))
   )
-  (hierarchical_label "RD" (shape input) (at 143.002 148.59 0)
+  (hierarchical_label "RD" (shape input) (at 144.526 148.59 0)
     (effects (font (size 1.27 1.27)) (justify left))
   )
@@
     (effects (font (size 1.27 1.27)) (justify right))
   )
-  (hierarchical_label "WR" (shape input) (at 142.748 146.05 0)
+  (hierarchical_label "WR" (shape input) (at 144.526 146.05 0)
     (effects (font (size 1.27 1.27)) (justify left))
   )
@@
     (effects (font (size 1.27 1.27)) (justify left))
   )
-  (hierarchical_label "HLDA" (shape input) (at 69.85 77.47 180)
-    (effects (font (size 1.27 1.27)) (justify right))
-  )
   (hierarchical_label "VCC" (shape input) (at 87.63 26.67 90)
     (effects (font (size 1.27 1.27)) (justify left))
@@
     (effects (font (size 1.27 1.27)) (justify right))
   )
-  (hierarchical_label "INTA" (shape input) (at 105.41 110.49 270)
+  (hierarchical_label "INTA" (shape input) (at 105.41 115.824 180)
     (effects (font (size 1.27 1.27)) (justify right))
   )
@@
     (effects (font (size 1.27 1.27)) (justify left))
   )
-  (hierarchical_label "HOLD" (shape input) (at 69.85 82.55 180)
-    (effects (font (size 1.27 1.27)) (justify right))
-  )
   (hierarchical_label "VCC" (shape input) (at 214.63 33.02 90)
     (effects (font (size 1.27 1.27)) (justify left))
@@
     (effects (font (size 1.27 1.27)) (justify left))
   )
-  (hierarchical_label "M{slash}IO" (shape input) (at 142.748 143.51 0)
+  (hierarchical_label "M{slash}IO" (shape input) (at 144.272 143.51 0)
     (effects (font (size 1.27 1.27)) (justify left))
   )

Commit message: stuff
Parts:
- added C12: 0.1uF, symbol Device:C
Connections:
- net GND: now also U1.30 (HLDA), U1.31 (HOLD), C12.1
- net VCC: now also U1.23 (~{TEST}), C12.2
- no-connect marks 14 -> 11
Changed lines of the file:
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@@
   (junction (at 121.92 176.53) (diameter 0) (color 0 0 0 0)
   )
+  (junction (at 69.85 82.55) (diameter 0) (color 0 0 0 0)
+  )
   (junction (at 55.118 52.07) (diameter 0) (color 0 0 0 0)
   )
@@
   (junction (at 198.12 63.5) (diameter 0) (color 0 0 0 0)
   )
+  (junction (at 87.63 22.86) (diameter 0) (color 0 0 0 0)
+  )
   (junction (at 109.22 168.91) (diameter 0) (color 0 0 0 0)
   )
   (junction (at 151.13 107.95) (diameter 0) (color 0 0 0 0)
   )
-  (no_connect (at 69.85 64.77))
   (no_connect (at 134.62 156.21))
   (no_connect (at 134.62 151.13))
   (no_connect (at 134.62 153.67))
-  (no_connect (at 69.85 82.55))
-  (no_connect (at 69.85 77.47))
   (no_connect (at 180.34 146.05))
   (no_connect (at 205.74 140.97))
@@
     (stroke (width 0) (type default) (color 0 0 0 0))
   )
+  (wire (pts (xy 69.85 82.55) (xy 69.85 87.63))
+    (stroke (width 0) (type default) (color 0 0 0 0))
+  )
   (wire (pts (xy 162.56 48.26) (xy 165.1 48.26))
     (stroke (width 0) (type default) (color 0 0 0 0))
@@
     (stroke (width 0) (type default) (color 0 0 0 0))
   )
+  (wire (pts (xy 87.63 20.32) (xy 87.63 22.86))
+    (stroke (width 0) (type default) (color 0 0 0 0))
+  )
   (wire (pts (xy 261.62 49.784) (xy 263.906 49.784))
     (stroke (width 0) (type default) (color 0 0 0 0))
@@
     (stroke (width 0) (type default) (color 0 0 0 0))
   )
+  (wire (pts (xy 87.63 22.86) (xy 87.63 26.67))
+    (stroke (width 0) (type default) (color 0 0 0 0))
+  )
   (bus (pts (xy 259.08 136.652) (xy 259.08 134.112))
     (stroke (width 0) (type default) (color 0 0 0 0))
@@
   )
   (bus (pts (xy 259.08 39.624) (xy 259.08 37.084))
+    (stroke (width 0) (type default) (color 0 0 0 0))
+  )
+  (wire (pts (xy 69.85 77.47) (xy 69.85 82.55))
     (stroke (width 0) (type default) (color 0 0 0 0))
   )
@@
     (effects (font (size 1.27 1.27)) (justify left))
   )
-  (hierarchical_label "VCC" (shape input) (at 87.63 26.67 90)
+  (hierarchical_label "VCC" (shape input) (at 87.63 20.32 90)
     (effects (font (size 1.27 1.27)) (justify left))
   )
@@
     (effects (font (size 1.27 1.27)) (justify left))
   )
+  (hierarchical_label "VCC" (shape input) (at 69.85 64.77 180)
+    (effects (font (size 1.27 1.27)) (justify right))
+  )
   (hierarchical_label "VCC" (shape input) (at 69.85 110.49 180)
     (effects (font (size 1.27 1.27)) (justify right))
@@
   (hierarchical_label "A[0..19]" (shape input) (at 167.64 44.958 0)
     (effects (font (size 1.27 1.27)) (justify left))
+  )
+  (symbol (lib_id "power:GND") (at 80.01 22.86 0) (unit 1)
+    (in_bom yes) (on_board yes) (fields_autoplaced)
+    (property "Reference" "#PWR0113" (id 0) (at 80.01 29.21 0)
+      (effects (font (size 1.27 1.27)) hide)
+    )
+    (property "Value" "GND" (id 1) (at 80.01 27.94 0))
+    (property "Footprint" "" (id 2) (at 80.01 22.86 0)
+      (effects (font (size 1.27 1.27)) hide)
+    )
+    (property "Datasheet" "" (id 3) (at 80.01 22.86 0)
+      (effects (font (size 1.27 1.27)) hide)
+    )
+    (pin "1")
   )
   (symbol (lib_id "Device:C") (at 55.118 55.88 0) (unit 1)
@@
     (pin "1")
   )
+  (symbol (lib_id "power:GND") (at 69.85 87.63 0) (unit 1)
+    (in_bom yes) (on_board yes) (fields_autoplaced)
+    (property "Reference" "#PWR0102" (id 0) (at 69.85 93.98 0)
+      (effects (font (size 1.27 1.27)) hide)
+    )
+    (property "Value" "" (id 1) (at 69.85 92.71 0))
+    (property "Footprint" "" (id 2) (at 69.85 87.63 0)
+      (effects (font (size 1.27 1.27)) hide)
+    )
+    (property "Datasheet" "" (id 3) (at 69.85 87.63 0)
+      (effects (font (size 1.27 1.27)) hide)
+    )
+    (pin "1")
+  )
   (symbol (lib_id "power:GND") (at 87.63 120.65 0) (unit 1)
     (in_bom yes) (on_board yes) (fields_autoplaced)
@@
     (pin "1")
   )
+  (symbol (lib_id "Device:C") (at 83.82 22.86 90) (unit 1)
+    (in_bom yes) (on_board yes) (fields_autoplaced)
+    (property "Reference" "C12" (id 0) (at 83.82 15.24 90))
+    (property "Value" "0.1uF" (id 1) (at 83.82 17.78 90))
+    (property "Footprint" "" (id 2) (at 87.63 21.8948 0)
+      (effects (font (size 1.27 1.27)) hide)
+    )
+    (property "Datasheet" "~" (id 3) (at 83.82 22.86 0)
+      (effects (font (size 1.27 1.27)) hide)
+    )
+    (pin "1")
+    (pin "2")
+  )
   (symbol (lib_id "power:GND") (at 149.86 76.2 0) (unit 1)

Commit message: finished design
Parts:
- C11: value 0.1uF -> 10uF; footprint (none) -> Capacitor_THT:C_Axial_L3.8mm_D2.6mm_P7.50mm_Horizontal
- C12: footprint (none) -> Capacitor_THT:C_Axial_L3.8mm_D2.6mm_P7.50mm_Horizontal
- J1: footprint (none) -> Connector_PinHeader_1.00mm:PinHeader_1x20_P1.00mm_Vertical
- J2: footprint (none) -> Connector_PinHeader_1.00mm:PinHeader_1x16_P1.00mm_Vertical
- J3: footprint (none) -> Connector_PinHeader_1.00mm:PinHeader_1x03_P1.00mm_Vertical
- R11: footprint (none) -> Resistor_THT:R_Axial_DIN0204_L3.6mm_D1.6mm_P1.90mm_Vertical
- SW0: footprint Audio_Module:Reverb_BTDR-1H -> Button_Switch_THT:SW_Tactile_Straight_KSA0Axx1LFTR
- U2, U3, U4, U5, U6, U7: footprint (none) -> Package_DIP:DIP-20_W7.62mm
Connections:
- net GND: no longer U1.30 (HLDA)
- no-connect marks 11 -> 12
Other:
- moved on the sheet: C11, C12, J1, J2, J3, R11, SW0, U1, U2, U3, U4, U5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
