File: Clock.kicad_sch (KiCad schematic)
At the start: 6 parts, among them SW1 SW_DIP_x01, U41 8284, Y1 Crystal

Commit message: stuff
Connections:
- net GND: now also U41.2 (PCLK)
- no-connect marks 8 -> 7
Other:
- moved on the sheet: C1, D1, R1, SW1, U41, Y1

Commit message: finished design
Parts:
- removed C1: 10uF, symbol pspice:CAP
- removed D1: DIODE, symbol pspice:DIODE
- removed R1: 10K, symbol Device:R
- removed SW1: SW_DIP_x01, symbol Switch:SW_DIP_x01
- added C41: 0.1uF, Capacitor_THT:C_Axial_L3.8mm_D2.6mm_P7.50mm_Horizontal, symbol Device:C
- added C42: 10uF, Capacitor_THT:C_Axial_L3.8mm_D2.6mm_P7.50mm_Horizontal, symbol Device:C
- added R41: 10k, Resistor_THT:R_Axial_DIN0204_L3.6mm_D1.6mm_P1.90mm_Vertical, symbol Device:R
- added SW41: SW_Push, Button_Switch_THT:SW_Tactile_Straight_KSA0Axx1LFTR, symbol Switch:SW_Push
- Y1: value Crystal -> 15MHZ; footprint (none) -> Crystal:Crystal_AT310_D3.0mm_L10.0mm_Vertical
Connections:
- net GND: now also U41.4 (RDY1), U41.6 (RDY2), C41.1, C42.2, SW41.1; no longer U41.2 (PCLK)
- net VCC: now also U41.15 (~{ASYNC}), U41.3 (~{AEN1}), U41.7 (~{AEN2}), C41.2, R41.1
- net at U41.11 (~{RES}): now also C42.1, R41.2, SW41.2
- new net PCLK: U41.2 (PCLK)
- no-connect marks 7 -> 2
