File: CMOS.kicad_sch (KiCad schematic)
At the start: 11 parts, among them U21 28F010, U210 74LS138, U211 74AUC2G04, U22 28F010, U23 28F010, U24 28F010, U25 28F010, U26 28F010, U27 28F010, U28 28F010, U29 74LS138

Commit message: stuff
Parts:
- removed U210, U29: 74LS138, symbol 74xx:74LS138
- removed U211: 74AUC2G04, symbol 74xGxx:74AUC2G04
- removed U23, U24, U25, U26, U27, U28: 28F010, parts:28F010, symbol 28F010:28F010
- added U23: 74LS138, symbol 74xx:74LS138
Connections:
- net A0: now also U23.3 (A2)
- net A18: now also U23.1 (A0)
- net A19: now also U23.2 (A1)
- net BHE: now also U23.5 (E2)
- net GND: now also U23.4 (E1), U23.8 (GND)
- net M/IO: now also U23.6 (E3)
- net VCC: now also U23.16 (VCC)
- net at U22.22 (CE): now also U21.22 (CE), U23.7 (O7)
- net MRDC renamed MRD
- net MWRC renamed MWR
- no-connect marks 16 -> 9
Other:
- moved on the sheet: U21

Commit message: finished design
Parts:
- added C21, C22: 0.1uF, Capacitor_THT:C_Axial_L3.8mm_D2.6mm_P7.50mm_Horizontal, symbol Device:C
- added U24: 74LS138, Package_DIP:DIP-16_W7.62mm, symbol 74xx:74LS138
- U23: footprint (none) -> Package_DIP:DIP-16_W7.62mm
Connections:
- net A0: now also U24.5 (E2); no longer U23.3 (A2)
- net A18: now also U24.1 (A0)
- net A19: now also U24.2 (A1)
- net GND: now also U23.3 (A2), C21.1, C22.1, U24.3 (A2), U24.4 (E1), U24.8 (GND)
- net M/IO: now also U24.6 (E3)
- net VCC: now also C21.2, C22.2, U24.16 (VCC)
- net at U23.12 (O3): now also U21.22 (CE)
- new net: U22.22 (CE), U24.7 (O7)
- now unconnected: U23.7 (O7)
- no-connect marks 9 -> 16
Other:
- moved on the sheet: U21, U22, U23

Commit message: yes
Connections:
- net D10: no longer U22.15 (DQ2)
- net D11: no longer U22.17 (DQ3)
- net D12: no longer U22.18 (DQ4)
- net D13: no longer U22.19 (DQ5)
- net D14: no longer U22.20 (DQ6)
- net D15: no longer U22.21 (DQ7)
- net D8: no longer U22.13 (DQ0)
- net D9: no longer U22.14 (DQ1)
- new net D0: U22.13 (DQ0)
- new net D1: U22.14 (DQ1)
- new net D2: U22.15 (DQ2)
- new net D3: U22.17 (DQ3)
- new net D4: U22.18 (DQ4)
- new net D5: U22.19 (DQ5)
- new net D6: U22.20 (DQ6)
- new net D7: U22.21 (DQ7)
Changed lines of the file:
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@@
-    (effects (font (size 1.27 1.27)) (justify left bottom))
-  )
-  (label "D10" (at 191.008 281.94 0)
     (effects (font (size 1.27 1.27)) (justify left bottom))
   )
@@
     (effects (font (size 1.27 1.27)) (justify left bottom))
   )
+  (label "D6" (at 191.568 271.78 0)
+    (effects (font (size 1.27 1.27)) (justify left bottom))
+  )
   (label "A7" (at 158.5437 64.7714 90)
+    (effects (font (size 1.27 1.27)) (justify left bottom))
+  )
+  (label "D4" (at 191.2622 276.86 0)
     (effects (font (size 1.27 1.27)) (justify left bottom))
   )
@@
     (effects (font (size 1.27 1.27)) (justify left bottom))
   )
+  (label "D1" (at 189.23 284.48 0)
+    (effects (font (size 1.27 1.27)) (justify left bottom))
+  )
   (label "D14" (at 191.008 115.57 0)
     (effects (font (size 1.27 1.27)) (justify left bottom))
@@
     (effects (font (size 1.27 1.27)) (justify left bottom))
   )
+  (label "D7" (at 191.1399 269.24 0)
+    (effects (font (size 1.27 1.27)) (justify left bottom))
+  )
   (label "A11" (at 168.6936 64.7713 90)
+    (effects (font (size 1.27 1.27)) (justify left bottom))
+  )
+  (label "D5" (at 191.3845 274.32 0)
     (effects (font (size 1.27 1.27)) (justify left bottom))
   )
@@
     (effects (font (size 1.27 1.27)) (justify left bottom))
   )
-  (label "D12" (at 191.008 276.86 0)
-    (effects (font (size 1.27 1.27)) (justify left bottom))
-  )
   (label "A10" (at 166.1489 220.9812 90)
     (effects (font (size 1.27 1.27)) (justify left bottom))
   )
   (label "A14" (at 176.3197 220.9814 90)
+    (effects (font (size 1.27 1.27)) (justify left bottom))
+  )
+  (label "D0" (at 189.23 287.02 0)
     (effects (font (size 1.27 1.27)) (justify left bottom))
   )
@@
     (effects (font (size 1.27 1.27)) (justify left bottom))
   )
-  (label "D13" (at 191.008 274.32 0)
-    (effects (font (size 1.27 1.27)) (justify left bottom))
-  )
   (label "A16" (at 181.3824 220.981 90)
     (effects (font (size 1.27 1.27)) (justify left bottom))
@@
     (effects (font (size 1.27 1.27)) (justify left bottom))
   )
-  (label "D9" (at 191.643 284.48 0)
+  (label "D3" (at 191.3233 279.4 0)
     (effects (font (size 1.27 1.27)) (justify left bottom))
   )
@@
     (effects (font (size 1.27 1.27)) (justify left bottom))
   )
-  (label "D15" (at 191.008 269.24 0)
+  (label "D2" (at 189.23 281.94 0)
     (effects (font (size 1.27 1.27)) (justify left bottom))
   )
@@
     (effects (font (size 1.27 1.27)) (justify left bottom))
   )
-  (label "D8" (at 191.643 287.02 0)
-    (effects (font (size 1.27 1.27)) (justify left bottom))
-  )
   (label "A13" (at 173.7638 64.771 90)
-    (effects (font (size 1.27 1.27)) (justify left bottom))
-  )
-  (label "D11" (at 191.008 279.4 0)
     (effects (font (size 1.27 1.27)) (justify left bottom))
   )
@@
     (effects (font (size 1.27 1.27)) (justify left bottom))
   )
-  (label "D14" (at 191.008 271.78 0)
-    (effects (font (size 1.27 1.27)) (justify left bottom))
-  )
