File: CMPE310_Final.kicad_pcb (KiCad board)
At the start: 6 copper layers, 182 parts, among them J1 Conn_01x20, J2 Conn_01x16, J3 Conn_01x03, J51 Conn_01x08, J52 Conn_01x08, J53 Conn_01x08, J61 Conn_01x04, J71 Conn_01x03, J72 Conn_01x02, J73 Conn_01x03, J91 DSUB-9, P1 Screw_Terminal_01x02, SW0 SW_Push, SW121 SW_DIP_x08, SW41 SW_Push, SW61 SW_Push, SW81 SW_Push, SW810 SW_Push, SW811 SW_Push, SW812 SW_Push, SW813 SW_Push, SW814 SW_Push, SW815 SW_Push, SW816 SW_Push, SW817 SW_Push, SW818 SW_Push, SW819 SW_Push, SW82 SW_Push, SW820 SW_Push, SW821 SW_Push, SW822 SW_Push, SW83 SW_Push, SW84 SW_Push, SW85 SW_Push, SW86 SW_Push, SW87 SW_Push, SW88 SW_Push, SW89 SW_Push, U1 8086_Min_Mode, U102 PAL16L8, U103 74LVC2G32, U104 74LVC2G32, U105 74LVC2G32, U111 74LS374, U1110 74LVC2G32, U1112 74LS374, U1113 HDSP-7401, U1115 74LS138, U1116 PAL16L8, U1117 74LVC2G32, U1118 74LVC2G32, U1119 74LVC2G32, U112 HDSP-7401, U1121 74LVC2G32, U1122 74LVC2G32, U115 PAL16L8, U116 74LS374, U117 74LVC2G32, U118 74LVC2G32, U119 74LVC2G32, U121 74AHC1G32, U122 74LS244, U123 PAL16L8, U124 74LVC2G32, U125 74LVC2G32, U126 74LVC2G32, U2 74AHC373, U21 28F010, U22 28F010, U23 74LS138, U24 74LS138, U3 74AHC373, U31 CY7C199, U32 74LS138, U33 CY7C199, U34 74LS138, U35 74LS138, U4 74AHC373, U41 8284, U5 74LS245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

Commit message: yes
Parts:
- removed R83: R, Resistor_THT:R_Axial_DIN0204_L3.6mm_D1.6mm_P1.90mm_Vertical
- U103, U104, U105, U1110, U1117, U1118, U1119, U1121, U1122, U117, U118, U119, U124, U125, U126, U57, U59, U63, U64, U65, U83, U84, U85: footprint Package_SO:SSOP-8_2.95x2.8mm_P0.65mm -> Package_DIP:DIP-8_W7.62mm
- U58: footprint Package_TO_SOT_SMD:SOT-23-5 -> Package_DIP:DIP-5-6_W7.62mm
- U73: footprint Package_TO_SOT_SMD:SOT-23-6 -> Package_DIP:DIP-6_W7.62mm
- moved C81 938.7 mm to (1055.2, 480.1), turned to 90 degrees
- moved U82 918.4 mm to (1023.6, 469.9), turned to 90 degrees
- moved U85 913.9 mm to (1050.3, 473.7), turned to -90 degrees
- moved U84 901.0 mm to (1047.8, 491.5), turned to 90 degrees
- moved U83 896.9 mm to (1037.6, 491.5), turned to 90 degrees
- moved U81 852.9 mm to (1051.6, 420.4), turned to 180 degrees
- moved SW83 666.8 mm to (1118.9, 477.7), turned to 180 degrees
- moved SW88 658.1 mm to (1118.9, 470.1), turned to 180 degrees
- moved SW84 650.4 mm to (1108.7, 477.7), turned to 180 degrees
- moved SW813 649.7 mm to (1118.9, 462.5), turned to 180 degrees
- moved SW89 641.5 mm to (1108.7, 470.1), turned to 180 degrees
- moved SW818 641.4 mm to (1118.9, 454.9), turned to 180 degrees
- moved U86 635.0 mm to (1116.3, 435.6), turned to -90 degrees
- moved SW85 634.2 mm to (1098.5, 477.7), turned to 180 degrees
- moved SW814 632.8 mm to (1108.7, 462.5), turned to 180 degrees
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Connections:
- U22 pad 13: D8 -> D0
- U22 pad 14: D9 -> D1
- U22 pad 15: D10 -> D2
- U22 pad 17: D11 -> D3
- U22 pad 18: D12 -> D4
- U22 pad 19: D13 -> D5
- U22 pad 20: D14 -> D6
- U22 pad 21: D15 -> D7
- U86 pad 6: Net-(R83-Pad1) -> VCC
Routing:
- net Net-(SW811-Pad2): track 0.00 -> 76.6 mm
- net Net-(SW812-Pad2): track 0.00 -> 76.4 mm
- net /8279 Bullet 8/RL1: track 0.00 -> 75.2 mm
- net /8279 Bullet 8/SL2: track 0.00 -> 73.7 mm
- net /8279 Bullet 8/RL0: track 0.00 -> 73.2 mm
- net /8279 Bullet 8/SL1: track 0.00 -> 71.8 mm
- net /8279 Bullet 8/SL0: track 0.00 -> 70.0 mm
- net Net-(SW810-Pad2): track 0.00 -> 68.9 mm
- net Net-(U81-Pad22): track 0.00 -> 65.4 mm
- net Net-(SW814-Pad2): track 0.00 -> 63.7 mm
- net Net-(SW813-Pad2): track 0.00 -> 63.5 mm
- net /8279 Bullet 8/RL3: track 0.00 -> 61.0 mm
- net /8279 Bullet 8/RL2: track 0.00 -> 56.0 mm
- net Net-(SW81-Pad1): track 0.00 -> 44.7 mm
- net Net-(SW82-Pad1): track 0.00 -> 38.9 mm
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