File: 8254.kicad_sch (KiCad schematic)
At the start: 1 part

Commit message: finished design
Parts:
- removed U?: (no value), symbol Timer:8254
- added C71: 0.1uF, Capacitor_THT:C_Axial_L3.8mm_D2.6mm_P7.50mm_Horizontal, symbol Device:C
- added J71, J73: Conn_01x03, Connector_PinHeader_1.00mm:PinHeader_1x03_P1.00mm_Vertical, symbol Connector_Generic:Conn_01x03
- added J72: Conn_01x02, Connector_PinHeader_1.00mm:PinHeader_1x02_P1.00mm_Vertical, symbol Connector_Generic:Conn_01x02
- added U71: 8254, Package_DIP:DIP-24_W15.24mm, symbol Timer:8254
- added U72: PAL16L8, Package_DIP:DIP-20_W7.62mm, symbol Logic_Programmable:PAL16L8
- added U73: 74LVC1G332, Package_TO_SOT_SMD:SOT-23-6, symbol 74xGxx:74LVC1G332
Connections:
- new net: J73.1 (Pin_1), U71.18 (CLK2)
- new net: J73.2 (Pin_2), U71.16 (G2)
- new net: J73.3 (Pin_3), U71.17 (OUT2)
- new net: U72.11 (I10), U73.4
- new net: U71.21 (~{CS}), U72.19 (IO1)
- new net: J71.3 (Pin_3), U71.10 (OUT0)
- new net: J71.2 (Pin_2), U71.11 (G0)
- new net: J72.2 (Pin_2), U71.14 (G1)
- new net: J72.1 (Pin_1), U71.15 (CLK1)
- new net: J71.1 (Pin_1), U71.9 (CLK0)
- new net A0: U72.2 (I2)
- new net A1: U71.19 (A0)
- new net A10: U72.12 (IO8)
- new net A11: U72.13 (IO7)
- new net A12: U72.14 (IO6)
- new net A13: U72.15 (IO5)
- new net A14: U72.16 (IO4)
- new net A15: U72.17 (I03)
- new net A16: U72.18 (IO2)
- new net A17: U73.6
- new net A18: U73.1
- new net A19: U73.3
- new net A2: U71.20 (A1)
- new net A3: U72.3 (I3)
- new net A4: U72.4 (I4)
- new net A5: U72.5 (I5)
- new net A6: U72.6 (I6)
- new net A7: U72.7 (I7)
- new net A8: U72.8 (I8)
- new net A9: U72.9 (I9)
- new net D0: U71.8 (D0)
- new net D1: U71.7 (D1)
- new net D2: U71.6 (D2)
- new net D3: U71.5 (D3)
- new net D4: U71.4 (D4)
- new net D5: U71.3 (D5)
- new net D6: U71.2 (D6)
- new net D7: U71.1 (D7)
- new net GND: C71.1, U71.12 (GND), U72.10 (GND), U73.2 (GND)
- new net IORD: U71.22 (~{RD})
- new net IOWR: U71.23 (~{WR})
- new net M/IO: U72.1 (I1)
- new net OUT1: U71.13 (OUT1)
- new net VCC: C71.2, U71.24 (VCC), U72.20 (VCC), U73.5 (VCC)
Other:
- note added: ";pins 1 2 3 4 5 6 7 8 9 10 M/IO A2 A3 A4 A5 A6 A7 A8 OR GND ;pins 11 12 13 14 15 16 17 18 19 20 A9 A10 A11 A12 A13 A14 A15 A16 O1 VCC Equation: /O1 = /M/IO * /OR * /A16 * A15 * A14 * A13 * A12 * A11 * A10 * A9 * A8 * A7 * A6 * /A5 * A4 * A3 * /A0"

Commit message: yes
Parts:
- U73: footprint Package_TO_SOT_SMD:SOT-23-6 -> (none)
Changed lines of the file:
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@@
     (property "Reference" "U73" (id 0) (at 57.8799 173.1531 0))
     (property "Value" "74LVC1G332" (id 1) (at 57.8799 175.6931 0))
-    (property "Footprint" "Package_TO_SOT_SMD:SOT-23-6" (id 2) (at 58.1262 167.6381 0)
+    (property "Footprint" "" (id 2) (at 58.1262 167.6381 0)
       (effects (font (size 1.27 1.27)) hide)
     )

Commit message: Finished
Parts:
- U73: footprint (none) -> Package_DIP:DIP-6_W7.62mm
Changed lines of the file:
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@@
     (property "Reference" "U73" (id 0) (at 57.8799 173.1531 0))
     (property "Value" "74LVC1G332" (id 1) (at 57.8799 175.6931 0))
-    (property "Footprint" "" (id 2) (at 58.1262 167.6381 0)
+    (property "Footprint" "Package_DIP:DIP-6_W7.62mm" (id 2) (at 58.1262 167.6381 0)
       (effects (font (size 1.27 1.27)) hide)
     )
