File: 8255.kicad_sch (KiCad schematic)
At the start: 11 parts, among them J51 Conn_01x08, J52 Conn_01x08, J53 Conn_01x08, U51 8255, U52 PAL16L8, U53 8255, U54 PAL16L8, U55 8255, U56 PAL16L8, U57 74AHC2G00, U59 74AHC2G00

Commit message: finished design
Parts:
- added C51, C52, C53: 0.1uF, Capacitor_THT:C_Axial_L3.8mm_D2.6mm_P7.50mm_Horizontal, symbol Device:C
- added U58: 74LVC1G32, Package_TO_SOT_SMD:SOT-23-5, symbol 74xGxx:74LVC1G32
- J51, J52, J53: footprint (none) -> Connector_PinHeader_1.00mm:PinHeader_1x08_P1.00mm_Vertical
- U52, U54, U56: footprint (none) -> Package_DIP:DIP-20_W7.62mm
- U57, U59: footprint (none) -> Package_SO:SSOP-8_2.95x2.8mm_P0.65mm
Connections:
- net A0: now also U58.2; no longer U53.6 (~{CS}), U54.19 (IO1)
- net GND: now also C51.1, C52.1, C53.1, U58.3 (GND)
- net VCC: now also C51.2, C52.2, C53.2, U58.5 (VCC)
- new net: U54.19 (IO1), U58.1
- new net: U53.6 (~{CS}), U58.4

Commit message: yes
Parts:
- U57, U59: footprint Package_SO:SSOP-8_2.95x2.8mm_P0.65mm -> (none)
- U58: footprint Package_TO_SOT_SMD:SOT-23-5 -> (none)
Changed lines of the file:
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@@
     (property "Reference" "U59" (id 0) (at 266.065 81.28 0))
     (property "Value" "74AHC2G00" (id 1) (at 266.065 83.82 0))
-    (property "Footprint" "Package_SO:SSOP-8_2.95x2.8mm_P0.65mm" (id 2) (at 266.7 89.154 0)
+    (property "Footprint" "" (id 2) (at 266.7 89.154 0)
       (effects (font (size 1.27 1.27)) hide)
     )
@@
     (property "Reference" "U57" (id 0) (at 90.043 36.83 0))
     (property "Value" "74AHC2G00" (id 1) (at 90.043 39.37 0))
-    (property "Footprint" "Package_SO:SSOP-8_2.95x2.8mm_P0.65mm" (id 2) (at 90.678 45.212 0)
+    (property "Footprint" "" (id 2) (at 90.678 45.212 0)
       (effects (font (size 1.27 1.27)) hide)
     )
@@
     (property "Reference" "U58" (id 0) (at 79.8671 144.78 0))
     (property "Value" "74LVC1G32" (id 1) (at 79.8671 147.32 0))
-    (property "Footprint" "Package_TO_SOT_SMD:SOT-23-5" (id 2) (at 80.5021 152.654 0)
-      (effects (font (size 1.27 1.27)) hide)
-    )
+    (property "Footprint" "" (id 2) (at 80.5021 152.654 0)
+      (effects (font (size 1.27 1.27)) hide)
+    )

Commit message: Finished
Parts:
- U57, U59: footprint (none) -> Package_DIP:DIP-8_W7.62mm
- U58: footprint (none) -> Package_DIP:DIP-5-6_W7.62mm
Changed lines of the file:
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@@
     (property "Reference" "U59" (id 0) (at 266.065 81.28 0))
     (property "Value" "74AHC2G00" (id 1) (at 266.065 83.82 0))
-    (property "Footprint" "" (id 2) (at 266.7 89.154 0)
+    (property "Footprint" "Package_DIP:DIP-8_W7.62mm" (id 2) (at 266.7 89.154 0)
       (effects (font (size 1.27 1.27)) hide)
     )
@@
     (property "Reference" "U57" (id 0) (at 90.043 36.83 0))
     (property "Value" "74AHC2G00" (id 1) (at 90.043 39.37 0))
-    (property "Footprint" "" (id 2) (at 90.678 45.212 0)
+    (property "Footprint" "Package_DIP:DIP-8_W7.62mm" (id 2) (at 90.678 45.212 0)
       (effects (font (size 1.27 1.27)) hide)
     )
@@
     (property "Reference" "U58" (id 0) (at 79.8671 144.78 0))
     (property "Value" "74LVC1G32" (id 1) (at 79.8671 147.32 0))
-    (property "Footprint" "" (id 2) (at 80.5021 152.654 0)
-      (effects (font (size 1.27 1.27)) hide)
-    )
+    (property "Footprint" "Package_DIP:DIP-5-6_W7.62mm" (id 2) (at 80.5021 152.654 0)
+      (effects (font (size 1.27 1.27)) hide)
+    )
