File: 8279.kicad_sch (KiCad schematic)
At the start: 30 parts, among them SW81 SW_Push, SW810 SW_Push, SW811 SW_Push, SW812 SW_Push, SW813 SW_Push, SW814 SW_Push, SW815 SW_Push, SW816 SW_Push, SW817 SW_Push, SW818 SW_Push, SW819 SW_Push, SW82 SW_Push, SW820 SW_Push, SW821 SW_Push, SW822 SW_Push, SW83 SW_Push, SW84 SW_Push, SW85 SW_Push, SW86 SW_Push, SW87 SW_Push, SW88 SW_Push, SW89 SW_Push, U81 pkd8279, U82 PAL16L8, U83 74LVC2G32, U84 74LVC2G32, U85 74LVC2G32, U86 74LS138

Commit message: yes
Parts:
- removed R83: R, Resistor_THT:R_Axial_DIN0204_L3.6mm_D1.6mm_P1.90mm_Vertical, symbol Device:R
- U83, U84, U85: footprint Package_SO:SSOP-8_2.95x2.8mm_P0.65mm -> (none)
Connections:
- net VCC: now also U86.6 (E3)
Changed lines of the file:
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@@
-    (stroke (width 0) (type default) (color 0 0 0 0))
-  )
-  (wire (pts (xy 201.168 139.192) (xy 201.168 122.428))
     (stroke (width 0) (type default) (color 0 0 0 0))
   )
@@
     (effects (font (size 1.27 1.27)) (justify right))
   )
-  (hierarchical_label "VCC" (shape input) (at 193.548 139.192 180)
+  (hierarchical_label "VCC" (shape input) (at 201.168 122.428 270)
     (effects (font (size 1.27 1.27)) (justify right))
   )
@@
     (property "Reference" "U85" (id 0) (at 52.4028 163.068 0))
     (property "Value" "74LVC2G32" (id 1) (at 52.4028 165.608 0))
-    (property "Footprint" "Package_SO:SSOP-8_2.95x2.8mm_P0.65mm" (id 2) (at 53.0378 170.3701 0)
+    (property "Footprint" "" (id 2) (at 53.0378 170.3701 0)
       (effects (font (size 1.27 1.27)) hide)
     )
@@
     (pin "2")
   )
-  (symbol (lib_id "Device:R") (at 197.358 139.192 270) (unit 1)
-    (in_bom yes) (on_board yes)
-    (property "Reference" "R83" (id 0) (at 197.358 132.588 90))
-    (property "Value" "R" (id 1) (at 197.358 135.128 90))
-    (property "Footprint" "Resistor_THT:R_Axial_DIN0204_L3.6mm_D1.6mm_P1.90mm_Vertical" (id 2) (at 197.358 137.414 90)
-      (effects (font (size 1.27 1.27)) hide)
-    )
-    (property "Datasheet" "~" (id 3) (at 197.358 139.192 0)
-      (effects (font (size 1.27 1.27)) hide)
-    )
-    (pin "1")
-    (pin "2")
-  )
   (symbol (lib_id "Switch:SW_Push") (at 220.472 57.7986 0) (unit 1)
     (in_bom yes) (on_board yes) (fields_autoplaced)
@@
     (property "Reference" "U83" (id 0) (at 38.4328 157.988 0))
     (property "Value" "74LVC2G32" (id 1) (at 38.4328 160.528 0))
-    (property "Footprint" "Package_SO:SSOP-8_2.95x2.8mm_P0.65mm" (id 2) (at 39.0678 166.3061 0)
+    (property "Footprint" "" (id 2) (at 39.0678 166.3061 0)
       (effects (font (size 1.27 1.27)) hide)
     )
@@
     (property "Reference" "U84" (id 0) (at 38.8138 179.2601 0))
     (property "Value" "74LVC2G32" (id 1) (at 38.8138 181.8001 0))
-    (property "Footprint" "Package_SO:SSOP-8_2.95x2.8mm_P0.65mm" (id 2) (at 38.8138 174.9421 0)
-      (effects (font (size 1.27 1.27)) hide)
-    )
+    (property "Footprint" "" (id 2) (at 38.8138 174.9421 0)
+      (effects (font (size 1.27 1.27)) hide)
+    )

Commit message: Finished
Parts:
- U83, U84, U85: footprint (none) -> Package_DIP:DIP-8_W7.62mm
Changed lines of the file:
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@@
     (property "Reference" "U85" (id 0) (at 52.4028 163.068 0))
     (property "Value" "74LVC2G32" (id 1) (at 52.4028 165.608 0))
-    (property "Footprint" "" (id 2) (at 53.0378 170.3701 0)
+    (property "Footprint" "Package_DIP:DIP-8_W7.62mm" (id 2) (at 53.0378 170.3701 0)
       (effects (font (size 1.27 1.27)) hide)
     )
@@
     (property "Reference" "U83" (id 0) (at 38.4328 157.988 0))
     (property "Value" "74LVC2G32" (id 1) (at 38.4328 160.528 0))
-    (property "Footprint" "" (id 2) (at 39.0678 166.3061 0)
+    (property "Footprint" "Package_DIP:DIP-8_W7.62mm" (id 2) (at 39.0678 166.3061 0)
       (effects (font (size 1.27 1.27)) hide)
     )
@@
     (property "Reference" "U84" (id 0) (at 38.8138 179.2601 0))
     (property "Value" "74LVC2G32" (id 1) (at 38.8138 181.8001 0))
-    (property "Footprint" "" (id 2) (at 38.8138 174.9421 0)
-      (effects (font (size 1.27 1.27)) hide)
-    )
+    (property "Footprint" "Package_DIP:DIP-8_W7.62mm" (id 2) (at 38.8138 174.9421 0)
+      (effects (font (size 1.27 1.27)) hide)
+    )
