File: CMPE310_Final.kicad_sch (KiCad schematic)
At the start: 1 part

Commit message: Added Second Resistor
Parts:
- added R?: R, symbol Device:R
Changed lines of the file:
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@@
 (kicad_sch (version 20211123) (generator eeschema)
   (paper "A4")
+  (symbol (lib_id "Device:R") (at 162.56 86.36 0) (unit 1)
+    (in_bom yes) (on_board yes) (fields_autoplaced)
+    (property "Reference" "R?" (id 0) (at 165.1 85.0899 0)
+      (effects (font (size 1.27 1.27)) (justify left))
+    )
+    (property "Value" "R" (id 1) (at 165.1 87.6299 0)
+      (effects (font (size 1.27 1.27)) (justify left))
+    )
+    (property "Footprint" "" (id 2) (at 160.782 86.36 90)
+      (effects (font (size 1.27 1.27)) hide)
+    )
+    (property "Datasheet" "~" (id 3) (at 162.56 86.36 0)
+      (effects (font (size 1.27 1.27)) hide)
+    )
+    (pin "1")
+    (pin "2")
+  )
   (symbol (lib_id "Device:R") (at 147.32 85.09 0) (unit 1)
     (in_bom yes) (on_board yes) (fields_autoplaced)
@@
   )
   (symbol_instances
+    (path "/1bd80cf9-f42a-4aee-a408-9dbf4e81e625"
+      (reference "R?") (unit 1) (value "R") (footprint "")
+    )
     (path "/e2eb2cd9-9b45-4dbc-b649-963ec3bf20f3"
       (reference "R?") (unit 1) (value "R") (footprint "")

Commit message: Added stuff
Parts:
- removed R? (x2): R, symbol Device:R
Changed lines of the file:
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@@
 (kicad_sch (version 20211123) (generator eeschema)
   (paper "A4")
-  (symbol (lib_id "Device:R") (at 162.56 86.36 0) (unit 1)
-    (in_bom yes) (on_board yes) (fields_autoplaced)
-    (property "Reference" "R?" (id 0) (at 165.1 85.0899 0)
-      (effects (font (size 1.27 1.27)) (justify left))
-    )
-    (property "Value" "R" (id 1) (at 165.1 87.6299 0)
-      (effects (font (size 1.27 1.27)) (justify left))
-    )
-    (property "Footprint" "" (id 2) (at 160.782 86.36 90)
-      (effects (font (size 1.27 1.27)) hide)
-    )
-    (property "Datasheet" "~" (id 3) (at 162.56 86.36 0)
-      (effects (font (size 1.27 1.27)) hide)
-    )
-    (pin "1")
-    (pin "2")
-  )
-  (symbol (lib_id "Device:R") (at 147.32 85.09 0) (unit 1)
-    (in_bom yes) (on_board yes) (fields_autoplaced)
-    (property "Reference" "R?" (id 0) (at 149.86 83.8199 0)
-      (effects (font (size 1.27 1.27)) (justify left))
-    )
-    (property "Value" "R" (id 1) (at 149.86 86.3599 0)
-      (effects (font (size 1.27 1.27)) (justify left))
-    )
-    (property "Footprint" "" (id 2) (at 145.542 85.09 90)
-      (effects (font (size 1.27 1.27)) hide)
-    )
-    (property "Datasheet" "~" (id 3) (at 147.32 85.09 0)
-      (effects (font (size 1.27 1.27)) hide)
-    )
-    (pin "1")
-    (pin "2")
-  )
   (sheet_instances
     (path "/" (page "1"))
   )
-  (symbol_instances
-    (path "/1bd80cf9-f42a-4aee-a408-9dbf4e81e625"
-      (reference "R?") (unit 1) (value "R") (footprint "")
-    )
-    (path "/e2eb2cd9-9b45-4dbc-b649-963ec3bf20f3"
-      (reference "R?") (unit 1) (value "R") (footprint "")
-    )
-  )
 )

Commit message: finished bullet 6
Parts:
- added C0: 100uF, symbol pspice:CAP
- added P1: Screw_Terminal_01x02, symbol Connector:Screw_Terminal_01x02
Connections:
- new net GND: C0.2, P1.2 (Pin_2)
- new net VCC: C0.1, P1.1 (Pin_1)
Other:
- added sheet 8086 Bullet One (8086 Bullet One.kicad_sch)
- added sheet 8255 Bullet 5 (8255.kicad_sch)
- added sheet 8259 Bullet 6 (8259.kicad_sch)
- added sheet CMOS Bullet Two (CMOS.kicad_sch)
- added sheet Clock Bullet Four (Clock.kicad_sch)
- added sheet SRAM Bullet Three (SRAM.kicad_sch)

Commit message: Added bullet 6
Connections:
- net VCC renamed +5V
Other:
- sheet 8086 Bullet One ports: added none; removed HLDA, HOLD
- sheet 8259 Bullet 6 ports: added none; removed Wait
- moved on the sheet: C0, P1

Commit message: stuff
Other:
- added sheet 8254 Bullet 7 (8254.kicad_sch)
- sheet 8259 Bullet 6 ports: added none; removed A[0..19], D[0..15], INT, INTA, IR1, IR2, IR3, M/IO, RD, VCC, WR
- sheet CMOS Bullet Two ports: added MRD, MWR; removed MRDC, MWRC
- sheet SRAM Bullet Three ports: added none; removed A[0..19], BHE, D[0..15], MRDC, MWTC, M/IO, VCC

Commit message: finished design
Parts:
- C0: footprint (none) -> Capacitor_THT:CP_Axial_L10.0mm_D4.5mm_P15.00mm_Horizontal
- P1: footprint (none) -> TerminalBlock:TerminalBlock_Altech_AK300-2_P5.00mm
Other:
- added sheet 8279 Bullet 8 (8279.kicad_sch)
- added sheet LCD Bullet 10 (LCD.kicad_sch)
- added sheet LED Bullet 11 (LED.kicad_sch)
- added sheet Switch bullet 12 (Switch.kicad_sch)
- added sheet UART Bullet 9 (UART.kicad_sch)
- sheet 8254 Bullet 7 ports: added A[0..19], D[0..15], IORD, IOWR, M/IO, OUT1, VCC; removed none
- sheet 8259 Bullet 6 ports: added A[0..19], D[0..15], INT, INTA, IR1, IR2, IR3, M/IO, RD, VCC, WR; removed none
- sheet Clock Bullet Four ports: added PCLK; removed none
- sheet SRAM Bullet Three ports: added A[0..19], BHE, D[0..15], MRD, MWR, M/IO, VCC; removed none
