File: LCD.kicad_sch (KiCad schematic)
At the start: 5 parts, among them U102 PAL16L8, U103 74LVC2G32, U104 74LVC2G32, U105 74LVC2G32

Commit message: yes
Parts:
- U103, U104, U105: footprint Package_SO:SSOP-8_2.95x2.8mm_P0.65mm -> (none)
Changed lines of the file:
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@@
     (property "Reference" "U105" (id 0) (at 89.2328 124.206 0))
     (property "Value" "74LVC2G32" (id 1) (at 89.2328 126.746 0))
-    (property "Footprint" "Package_SO:SSOP-8_2.95x2.8mm_P0.65mm" (id 2) (at 89.8678 132.2701 0)
+    (property "Footprint" "" (id 2) (at 89.8678 132.2701 0)
       (effects (font (size 1.27 1.27)) hide)
     )
@@
     (property "Reference" "U104" (id 0) (at 75.6438 141.1601 0))
     (property "Value" "74LVC2G32" (id 1) (at 75.6438 143.7001 0))
-    (property "Footprint" "Package_SO:SSOP-8_2.95x2.8mm_P0.65mm" (id 2) (at 75.6438 136.8421 0)
+    (property "Footprint" "" (id 2) (at 75.6438 136.8421 0)
       (effects (font (size 1.27 1.27)) hide)
     )
@@
     (property "Reference" "U103" (id 0) (at 75.2628 120.396 0))
     (property "Value" "74LVC2G32" (id 1) (at 75.2628 122.936 0))
-    (property "Footprint" "Package_SO:SSOP-8_2.95x2.8mm_P0.65mm" (id 2) (at 75.8978 128.2061 0)
+    (property "Footprint" "" (id 2) (at 75.8978 128.2061 0)
       (effects (font (size 1.27 1.27)) hide)
     )

Commit message: Finished
Parts:
- added C101: 0.1uF, Capacitor_THT:C_Axial_L3.8mm_D2.6mm_P7.50mm_Horizontal, symbol Device:C
- U103, U104, U105: footprint (none) -> Package_DIP:DIP-8_W7.62mm
Connections:
- net GND: now also DS101.1 (VSS), C101.1; no longer DS101.2 (VDD)
- net VCC: now also DS101.2 (VDD), C101.2; no longer DS101.1 (VSS)
Changed lines of the file:
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@@
   (junction (at 96.012 96.0187) (diameter 0) (color 0 0 0 0)
   )
-  (junction (at 152.5056 65.278) (diameter 0) (color 0 0 0 0)
+  (junction (at 152.5061 55.3288) (diameter 0) (color 0 0 0 0)
+  )
+  (junction (at 153.67 70.358) (diameter 0) (color 0 0 0 0)
   )
   (no_connect (at 181.61 88.138))
@@
     (stroke (width 0) (type default) (color 0 0 0 0))
   )
+  (wire (pts (xy 152.5061 54.864) (xy 152.5061 55.3288))
+    (stroke (width 0) (type default) (color 0 0 0 0))
+  )
   (wire (pts (xy 98.5958 111.76) (xy 102.108 111.76))
     (stroke (width 0) (type default) (color 0 0 0 0))
@@
     (stroke (width 0) (type default) (color 0 0 0 0))
   )
-  (wire (pts (xy 143.6867 67.818) (xy 153.67 67.818))
-    (stroke (width 0) (type default) (color 0 0 0 0))
-  )
   (wire (pts (xy 81.9938 133.5401) (xy 82.2478 133.5401))
     (stroke (width 0) (type default) (color 0 0 0 0))
@@
     (stroke (width 0) (type default) (color 0 0 0 0))
   )
-  (wire (pts (xy 143.6867 65.786) (xy 143.6867 67.818))
+  (wire (pts (xy 138.43 65.786) (xy 153.67 65.786))
     (stroke (width 0) (type default) (color 0 0 0 0))
   )
@@
     (stroke (width 0) (type default) (color 0 0 0 0))
   )
+  (wire (pts (xy 152.5061 65.2693) (xy 152.5056 65.2693))
+    (stroke (width 0) (type default) (color 0 0 0 0))
+  )
   (wire (pts (xy 98.5958 93.5081) (xy 98.552 72.898))
     (stroke (width 0) (type default) (color 0 0 0 0))
@@
     (stroke (width 0) (type default) (color 0 0 0 0))
   )
-  (wire (pts (xy 150.876 65.278) (xy 152.5056 65.278))
-    (stroke (width 0) (type default) (color 0 0 0 0))
-  )
   (bus (pts (xy 62.992 124.4786) (xy 62.992 127.0186))
     (stroke (width 0) (type default) (color 0 0 0 0))
@@
     (stroke (width 0) (type default) (color 0 0 0 0))
   )
+  (wire (pts (xy 152.5061 55.3288) (xy 152.5061 65.2693))
+    (stroke (width 0) (type default) (color 0 0 0 0))
+  )
   (wire (pts (xy 65.532 129.4761) (xy 65.532 129.5586))
     (stroke (width 0) (type default) (color 0 0 0 0))
@@
     (stroke (width 0) (type default) (color 0 0 0 0))
   )
+  (wire (pts (xy 153.67 67.818) (xy 153.67 70.358))
+    (stroke (width 0) (type default) (color 0 0 0 0))
+  )
+  (wire (pts (xy 148.336 54.864) (xy 152.5061 54.864))
+    (stroke (width 0) (type default) (color 0 0 0 0))
+  )
   (bus (pts (xy 62.992 129.5586) (xy 62.992 132.0161))
     (stroke (width 0) (type default) (color 0 0 0 0))
@@
     (stroke (width 0) (type default) (color 0 0 0 0))
   )
+  (wire (pts (xy 153.67 65.786) (xy 153.67 65.278))
+    (stroke (width 0) (type default) (color 0 0 0 0))
+  )
   (bus (pts (xy 96.0558 101.6) (xy 96.0558 104.14))
     (stroke (width 0) (type default) (color 0 0 0 0))
@@
     (stroke (width 0) (type default) (color 0 0 0 0))
   )
-  (wire (pts (xy 152.5056 70.358) (xy 152.5056 65.278))
+  (wire (pts (xy 152.5056 65.2693) (xy 152.5056 70.358))
     (stroke (width 0) (type default) (color 0 0 0 0))
   )
@@
   )
   (bus (pts (xy 96.0558 114.3) (xy 96.0558 116.84))
-    (stroke (width 0) (type default) (color 0 0 0 0))
-  )
-  (wire (pts (xy 138.43 65.786) (xy 143.6867 65.786))
-    (stroke (width 0) (type default) (color 0 0 0 0))
-  )
-  (wire (pts (xy 152.5056 65.278) (xy 153.67 65.278))
     (stroke (width 0) (type default) (color 0 0 0 0))
   )
@@
     (effects (font (size 1.27 1.27)) (justify left))
   )
-  (hierarchical_label "VCC" (shape input) (at 150.876 65.278 180)
+  (hierarchical_label "VCC" (shape input) (at 148.336 54.864 180)
     (effects (font (size 1.27 1.27)) (justify right))
   )
@@
     (property "Reference" "U105" (id 0) (at 89.2328 124.206 0))
     (property "Value" "74LVC2G32" (id 1) (at 89.2328 126.746 0))
-    (property "Footprint" "" (id 2) (at 89.8678 132.2701 0)
+    (property "Footprint" "Package_DIP:DIP-8_W7.62mm" (id 2) (at 89.8678 132.2701 0)
       (effects (font (size 1.27 1.27)) hide)
     )
@@
     (property "Reference" "U104" (id 0) (at 75.6438 141.1601 0))
     (property "Value" "74LVC2G32" (id 1) (at 75.6438 143.7001 0))
-    (property "Footprint" "" (id 2) (at 75.6438 136.8421 0)
+    (property "Footprint" "Package_DIP:DIP-8_W7.62mm" (id 2) (at 75.6438 136.8421 0)
       (effects (font (size 1.27 1.27)) hide)
     )
@@
     (pin "5")
     (pin "6")
+  )
+  (symbol (lib_id "power:GND") (at 160.1261 55.3288 0) (unit 1)
+    (in_bom yes) (on_board yes) (fields_autoplaced)
+    (property "Reference" "#PWR0188" (id 0) (at 160.1261 61.6788 0)
+      (effects (font (size 1.27 1.27)) hide)
+    )
+    (property "Value" "GND" (id 1) (at 160.1261 59.7842 0))
+    (property "Footprint" "" (id 2) (at 160.1261 55.3288 0)
+      (effects (font (size 1.27 1.27)) hide)
+    )
+    (property "Datasheet" "" (id 3) (at 160.1261 55.3288 0)
+      (effects (font (size 1.27 1.27)) hide)
+    )
+    (pin "1")
+  )
+  (symbol (lib_id "Device:C") (at 156.3161 55.3288 270) (unit 1)
+    (in_bom yes) (on_board yes) (fields_autoplaced)
+    (property "Reference" "C101" (id 0) (at 156.3161 48.26 90))
+    (property "Value" "0.1uF" (id 1) (at 156.3161 50.8 90))
+    (property "Footprint" "Capacitor_THT:C_Axial_L3.8mm_D2.6mm_P7.50mm_Horizontal" (id 2) (at 152.5061 56.294 0)
+      (effects (font (size 1.27 1.27)) hide)
+    )
+    (property "Datasheet" "~" (id 3) (at 156.3161 55.3288 0)
+      (effects (font (size 1.27 1.27)) hide)
+    )
+    (pin "1")
+    (pin "2")
   )
   (symbol (lib_id "Logic_Programmable:PAL16L8") (at 114.808 114.3 0) (unit 1)
@@
     (property "Reference" "U103" (id 0) (at 75.2628 120.396 0))
     (property "Value" "74LVC2G32" (id 1) (at 75.2628 122.936 0))
-    (property "Footprint" "" (id 2) (at 75.8978 128.2061 0)
-      (effects (font (size 1.27 1.27)) hide)
-    )
+    (property "Footprint" "Package_DIP:DIP-8_W7.62mm" (id 2) (at 75.8978 128.2061 0)
+      (effects (font (size 1.27 1.27)) hide)
+    )
