File: LED.kicad_sch (KiCad schematic)
At the start: 58 parts, among them U111 74LS374, U1110 74LVC2G32, U1112 74LS374, U1113 HDSP-7401, U1115 74LS138, U1116 PAL16L8, U1117 74LVC2G32, U1118 74LVC2G32, U1119 74LVC2G32, U112 HDSP-7401, U1121 74LVC2G32, U1122 74LVC2G32, U115 PAL16L8, U116 74LS374, U117 74LVC2G32, U118 74LVC2G32, U119 74LVC2G32

Commit message: yes
Parts:
- U1110, U1117, U1118, U1119, U1121, U1122, U117, U118, U119: footprint Package_SO:SSOP-8_2.95x2.8mm_P0.65mm -> (none)
Changed lines of the file:
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@@
     (property "Reference" "U1117" (id 0) (at 48.6677 134.874 0))
     (property "Value" "74LVC2G32" (id 1) (at 48.6677 137.414 0))
-    (property "Footprint" "Package_SO:SSOP-8_2.95x2.8mm_P0.65mm" (id 2) (at 49.3027 142.6841 0)
+    (property "Footprint" "" (id 2) (at 49.3027 142.6841 0)
       (effects (font (size 1.27 1.27)) hide)
     )
@@
     (property "Reference" "U118" (id 0) (at 200.4076 228.092 0))
     (property "Value" "74LVC2G32" (id 1) (at 200.4076 230.632 0))
-    (property "Footprint" "Package_SO:SSOP-8_2.95x2.8mm_P0.65mm" (id 2) (at 201.0426 235.9021 0)
+    (property "Footprint" "" (id 2) (at 201.0426 235.9021 0)
       (effects (font (size 1.27 1.27)) hide)
     )
@@
     (property "Reference" "U119" (id 0) (at 186.8186 244.7921 0))
     (property "Value" "74LVC2G32" (id 1) (at 186.8186 247.3321 0))
-    (property "Footprint" "Package_SO:SSOP-8_2.95x2.8mm_P0.65mm" (id 2) (at 186.8186 240.4741 0)
+    (property "Footprint" "" (id 2) (at 186.8186 240.4741 0)
       (effects (font (size 1.27 1.27)) hide)
     )
@@
     (property "Reference" "U1119" (id 0) (at 49.0487 155.6381 0))
     (property "Value" "74LVC2G32" (id 1) (at 49.0487 158.1781 0))
-    (property "Footprint" "Package_SO:SSOP-8_2.95x2.8mm_P0.65mm" (id 2) (at 49.0487 151.3201 0)
+    (property "Footprint" "" (id 2) (at 49.0487 151.3201 0)
       (effects (font (size 1.27 1.27)) hide)
     )
@@
     (property "Reference" "U117" (id 0) (at 186.4376 224.282 0))
     (property "Value" "74LVC2G32" (id 1) (at 186.4376 226.822 0))
-    (property "Footprint" "Package_SO:SSOP-8_2.95x2.8mm_P0.65mm" (id 2) (at 187.0726 231.8381 0)
+    (property "Footprint" "" (id 2) (at 187.0726 231.8381 0)
       (effects (font (size 1.27 1.27)) hide)
     )
@@
     (property "Reference" "U1122" (id 0) (at 150.6397 123.952 0))
     (property "Value" "74LVC2G32" (id 1) (at 150.6397 126.492 0))
-    (property "Footprint" "Package_SO:SSOP-8_2.95x2.8mm_P0.65mm" (id 2) (at 151.2747 131.826 0)
+    (property "Footprint" "" (id 2) (at 151.2747 131.826 0)
       (effects (font (size 1.27 1.27)) hide)
     )
@@
     (property "Reference" "U1121" (id 0) (at 144.1224 70.0277 0))
     (property "Value" "74LVC2G32" (id 1) (at 144.1224 72.5677 0))
-    (property "Footprint" "Package_SO:SSOP-8_2.95x2.8mm_P0.65mm" (id 2) (at 144.7574 77.805 0)
+    (property "Footprint" "" (id 2) (at 144.7574 77.805 0)
       (effects (font (size 1.27 1.27)) hide)
     )
@@
     (property "Reference" "U1118" (id 0) (at 62.6377 138.684 0))
     (property "Value" "74LVC2G32" (id 1) (at 62.6377 141.224 0))
-    (property "Footprint" "Package_SO:SSOP-8_2.95x2.8mm_P0.65mm" (id 2) (at 63.2727 146.7481 0)
+    (property "Footprint" "" (id 2) (at 63.2727 146.7481 0)
       (effects (font (size 1.27 1.27)) hide)
     )
@@
     (property "Reference" "U1110" (id 0) (at 247.6183 240.3444 0))
     (property "Value" "74LVC2G32" (id 1) (at 247.6183 242.8844 0))
-    (property "Footprint" "Package_SO:SSOP-8_2.95x2.8mm_P0.65mm" (id 2) (at 247.6183 236.0264 0)
-      (effects (font (size 1.27 1.27)) hide)
-    )
+    (property "Footprint" "" (id 2) (at 247.6183 236.0264 0)
+      (effects (font (size 1.27 1.27)) hide)
+    )

Commit message: Finished
Parts:
- U1110, U1117, U1118, U1119, U1121, U1122, U117, U118, U119: footprint (none) -> Package_DIP:DIP-8_W7.62mm
Changed lines of the file:
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@@
     (property "Reference" "U1117" (id 0) (at 48.6677 134.874 0))
     (property "Value" "74LVC2G32" (id 1) (at 48.6677 137.414 0))
-    (property "Footprint" "" (id 2) (at 49.3027 142.6841 0)
+    (property "Footprint" "Package_DIP:DIP-8_W7.62mm" (id 2) (at 49.3027 142.6841 0)
       (effects (font (size 1.27 1.27)) hide)
     )
@@
     (property "Reference" "U118" (id 0) (at 200.4076 228.092 0))
     (property "Value" "74LVC2G32" (id 1) (at 200.4076 230.632 0))
-    (property "Footprint" "" (id 2) (at 201.0426 235.9021 0)
+    (property "Footprint" "Package_DIP:DIP-8_W7.62mm" (id 2) (at 201.0426 235.9021 0)
       (effects (font (size 1.27 1.27)) hide)
     )
@@
     (property "Reference" "U119" (id 0) (at 186.8186 244.7921 0))
     (property "Value" "74LVC2G32" (id 1) (at 186.8186 247.3321 0))
-    (property "Footprint" "" (id 2) (at 186.8186 240.4741 0)
+    (property "Footprint" "Package_DIP:DIP-8_W7.62mm" (id 2) (at 186.8186 240.4741 0)
       (effects (font (size 1.27 1.27)) hide)
     )
@@
     (property "Reference" "U1119" (id 0) (at 49.0487 155.6381 0))
     (property "Value" "74LVC2G32" (id 1) (at 49.0487 158.1781 0))
-    (property "Footprint" "" (id 2) (at 49.0487 151.3201 0)
+    (property "Footprint" "Package_DIP:DIP-8_W7.62mm" (id 2) (at 49.0487 151.3201 0)
       (effects (font (size 1.27 1.27)) hide)
     )
@@
     (property "Reference" "U117" (id 0) (at 186.4376 224.282 0))
     (property "Value" "74LVC2G32" (id 1) (at 186.4376 226.822 0))
-    (property "Footprint" "" (id 2) (at 187.0726 231.8381 0)
+    (property "Footprint" "Package_DIP:DIP-8_W7.62mm" (id 2) (at 187.0726 231.8381 0)
       (effects (font (size 1.27 1.27)) hide)
     )
@@
     (property "Reference" "U1122" (id 0) (at 150.6397 123.952 0))
     (property "Value" "74LVC2G32" (id 1) (at 150.6397 126.492 0))
-    (property "Footprint" "" (id 2) (at 151.2747 131.826 0)
+    (property "Footprint" "Package_DIP:DIP-8_W7.62mm" (id 2) (at 151.2747 131.826 0)
       (effects (font (size 1.27 1.27)) hide)
     )
@@
     (property "Reference" "U1121" (id 0) (at 144.1224 70.0277 0))
     (property "Value" "74LVC2G32" (id 1) (at 144.1224 72.5677 0))
-    (property "Footprint" "" (id 2) (at 144.7574 77.805 0)
+    (property "Footprint" "Package_DIP:DIP-8_W7.62mm" (id 2) (at 144.7574 77.805 0)
       (effects (font (size 1.27 1.27)) hide)
     )
@@
     (property "Reference" "U1118" (id 0) (at 62.6377 138.684 0))
     (property "Value" "74LVC2G32" (id 1) (at 62.6377 141.224 0))
-    (property "Footprint" "" (id 2) (at 63.2727 146.7481 0)
+    (property "Footprint" "Package_DIP:DIP-8_W7.62mm" (id 2) (at 63.2727 146.7481 0)
       (effects (font (size 1.27 1.27)) hide)
     )
@@
     (property "Reference" "U1110" (id 0) (at 247.6183 240.3444 0))
     (property "Value" "74LVC2G32" (id 1) (at 247.6183 242.8844 0))
-    (property "Footprint" "" (id 2) (at 247.6183 236.0264 0)
-      (effects (font (size 1.27 1.27)) hide)
-    )
+    (property "Footprint" "Package_DIP:DIP-8_W7.62mm" (id 2) (at 247.6183 236.0264 0)
+      (effects (font (size 1.27 1.27)) hide)
+    )
