File: Switch.kicad_sch (KiCad schematic)
At the start: 16 parts, among them SW121 SW_DIP_x08, U121 74AHC1G32, U122 74LS244, U123 PAL16L8, U124 74LVC2G32, U125 74LVC2G32, U126 74LVC2G32

Commit message: yes
Parts:
- U124, U125, U126: footprint Package_SO:SSOP-8_2.95x2.8mm_P0.65mm -> (none)
Changed lines of the file:
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@@
     (property "Reference" "U126" (id 0) (at 104.2188 147.32 0))
     (property "Value" "74LVC2G32" (id 1) (at 104.2188 149.86 0))
-    (property "Footprint" "Package_SO:SSOP-8_2.95x2.8mm_P0.65mm" (id 2) (at 104.8538 155.3841 0)
+    (property "Footprint" "" (id 2) (at 104.8538 155.3841 0)
       (effects (font (size 1.27 1.27)) hide)
     )
@@
     (property "Reference" "U125" (id 0) (at 90.6298 164.2741 0))
     (property "Value" "74LVC2G32" (id 1) (at 90.6298 166.8141 0))
-    (property "Footprint" "Package_SO:SSOP-8_2.95x2.8mm_P0.65mm" (id 2) (at 90.6298 159.9561 0)
+    (property "Footprint" "" (id 2) (at 90.6298 159.9561 0)
       (effects (font (size 1.27 1.27)) hide)
     )
@@
     (property "Reference" "U124" (id 0) (at 90.2488 143.51 0))
     (property "Value" "74LVC2G32" (id 1) (at 90.2488 146.05 0))
-    (property "Footprint" "Package_SO:SSOP-8_2.95x2.8mm_P0.65mm" (id 2) (at 90.8838 151.3201 0)
+    (property "Footprint" "" (id 2) (at 90.8838 151.3201 0)
       (effects (font (size 1.27 1.27)) hide)
     )

Commit message: Finished
Parts:
- U124, U125, U126: footprint (none) -> Package_DIP:DIP-8_W7.62mm
Changed lines of the file:
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@@
     (property "Reference" "U126" (id 0) (at 104.2188 147.32 0))
     (property "Value" "74LVC2G32" (id 1) (at 104.2188 149.86 0))
-    (property "Footprint" "" (id 2) (at 104.8538 155.3841 0)
+    (property "Footprint" "Package_DIP:DIP-8_W7.62mm" (id 2) (at 104.8538 155.3841 0)
       (effects (font (size 1.27 1.27)) hide)
     )
@@
     (property "Reference" "U125" (id 0) (at 90.6298 164.2741 0))
     (property "Value" "74LVC2G32" (id 1) (at 90.6298 166.8141 0))
-    (property "Footprint" "" (id 2) (at 90.6298 159.9561 0)
+    (property "Footprint" "Package_DIP:DIP-8_W7.62mm" (id 2) (at 90.6298 159.9561 0)
       (effects (font (size 1.27 1.27)) hide)
     )
@@
     (property "Reference" "U124" (id 0) (at 90.2488 143.51 0))
     (property "Value" "74LVC2G32" (id 1) (at 90.2488 146.05 0))
-    (property "Footprint" "" (id 2) (at 90.8838 151.3201 0)
+    (property "Footprint" "Package_DIP:DIP-8_W7.62mm" (id 2) (at 90.8838 151.3201 0)
       (effects (font (size 1.27 1.27)) hide)
     )
