File: SRAM.kicad_sch (KiCad schematic)
At the start: 11 parts, among them U31 CY7C199, U310 CY7C199, U311 CY7C199, U312 CY7C199, U313 74LS138, U32 CY7C199, U33 CY7C199, U34 CY7C199, U35 74LS138, U36 74LS138, U39 CY7C199

Commit message: Added bullet 6
Changed lines of the file:
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@@
     (effects (font (size 1.27 1.27)) (justify left bottom))
   )
-  (label "A18" (at 25.1523 152.146 0)
+  (label "A18" (at 25.146 152.146 0)
     (effects (font (size 1.27 1.27)) (justify left bottom))
   )
@@
     (effects (font (size 1.27 1.27)) (justify left bottom))
   )
-  (label "A19" (at 25.1523 154.686 0)
-    (effects (font (size 1.27 1.27)) (justify left bottom))
-  )
+  (label "A19" (at 25.146 154.686 0)
+    (effects (font (size 1.27 1.27)) (justify left bottom))
+  )

Commit message: stuff
Parts:
- removed U310, U311, U312, U32, U33, U34: CY7C199, symbol Memory_RAM:CY7C199
- removed U313, U35, U36: 74LS138, symbol 74xx:74LS138
Connections:
- net MRDC: no longer names the net of U31.22 (~{OE})
- net MRDC: no longer U39.22 (~{OE})
- net MWTC: no longer names the net of U31.27 (~{WE})
- net MWTC: no longer U39.27 (~{WE})
- no-connect marks 15 -> 0
Other:
- moved on the sheet: U31, U39

Commit message: finished design
Parts:
- added C31, C32: 0.1uF, Capacitor_THT:C_Axial_L3.8mm_D2.6mm_P7.50mm_Horizontal, symbol Device:C
- added U32, U34, U35: 74LS138, Package_DIP:DIP-16_W7.62mm, symbol 74xx:74LS138
- U31: footprint (none) -> Package_DIP:DIP-28_W7.62mm
- U33: renamed from U39; footprint (none) -> Package_DIP:DIP-28_W7.62mm
Connections:
- net GND: now also C31.1, C32.1, U32.3 (A2), U32.8 (GND), U34.3 (A2), U34.8 (GND), U35.3 (A2), U35.4 (E1), U35.5 (E2), U35.8 (GND)
- net VCC: now also C31.2, C32.2, U32.16 (VCC), U34.16 (VCC), U35.16 (VCC), U35.6 (E3)
- net at U31.20 (~{CE}): now also U32.15 (O0)
- net MRD: now reaches U31.22 (~{OE})
- net MRD: now also U33.22 (~{OE})
- net MWR: now reaches U31.27 (~{WE})
- net MWR: now also U33.27 (~{WE})
- net at U33.20 (~{CE}): now also U34.15 (O0)
- new net: U32.4 (E1), U34.4 (E1), U35.15 (O0)
- new net A0: U34.5 (E2)
- new net A16: U32.1 (A0), U34.1 (A0)
- new net A17: U32.2 (A1), U34.2 (A1)
- new net A18: U35.1 (A0)
- new net A19: U35.2 (A1)
- new net BHE: U32.5 (E2)
- new net M/IO: U32.6 (E3), U34.6 (E3)
- no-connect marks 0 -> 21
Other:
- moved on the sheet: U31, U33

Commit message: Finished
Parts:
- added C1, C34: 0.1uF, Capacitor_THT:C_Axial_L3.8mm_D2.6mm_P7.50mm_Horizontal, symbol Device:C
- added U36, U37: CY7C199, Package_DIP:DIP-28_W7.62mm, symbol Memory_RAM:CY7C199
Connections:
- net A1: now also U36.21 (A0), U37.21 (A0)
- net A10: now also U36.5 (A9), U37.5 (A9)
- net A11: now also U36.6 (A10), U37.6 (A10)
- net A12: now also U36.7 (A11), U37.7 (A11)
- net A13: now also U36.8 (A12), U37.8 (A12)
- net A14: now also U36.9 (A13), U37.9 (A13)
- net A15: now also U36.10 (A14), U37.10 (A14)
- net A2: now also U36.23 (A1), U37.23 (A1)
- net A3: now also U36.24 (A2), U37.24 (A2)
- net A4: now also U36.25 (A3), U37.25 (A3)
- net A5: now also U36.26 (A4), U37.26 (A4)
- net A6: now also U36.1 (A5), U37.1 (A5)
- net A7: now also U36.2 (A6), U37.2 (A6)
- net A8: now also U36.3 (A7), U37.3 (A7)
- net A9: now also U36.4 (A8), U37.4 (A8)
- net D0: now also U37.11 (D0)
- net D1: now also U37.12 (D1)
- net D10: now also U36.13 (D2)
- net D11: now also U36.15 (D3)
- net D12: now also U36.16 (D4)
- net D13: now also U36.17 (D5)
- net D14: now also U36.18 (D6)
- net D15: now also U36.19 (D7)
- net D2: now also U37.13 (D2)
- net D3: now also U37.15 (D3)
- net D4: now also U37.16 (D4)
- net D5: now also U37.17 (D5)
- net D6: now also U37.18 (D6)
- net D7: now also U37.19 (D7)
- net D8: now also U36.11 (D0)
- net D9: now also U36.12 (D1)
- net GND: now also C1.1, C34.1, U36.14 (GND), U37.14 (GND)
- net MRD: now also U36.22 (~{OE}), U37.22 (~{OE})
- net MWR: now also U36.27 (~{WE}), U37.27 (~{WE})
- net VCC: now also C1.2, C34.2, U36.28 (VCC), U37.28 (VCC)
- net at U32.14 (O1): now also U36.20 (~{CE})
- net at U34.14 (O1): now also U37.20 (~{CE})
- no-connect marks 21 -> 19
